File: schematic/pslab-mini.kicad_sch (KiCad schematic)
At the start: 0 parts

Commit message: Update pslab-mini.kicad_sch
Other:
- title: PSLab-Mini -> PSLab-Mini-WR
Changed lines of the file:
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@@
 	(paper "A4")
 	(title_block
-		(title "PSLab-Mini")
+		(title "PSLab-Mini-WR")
 		(date "2025-07-16")
 		(rev "0.0.0")

Commit message: Update pslab-mini.kicad_sch
Other:
- title: PSLab-Mini-WR -> PSLab-Mini-WR2
Changed lines of the file:
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@@
 	(paper "A4")
 	(title_block
-		(title "PSLab-Mini-WR")
+		(title "PSLab-Mini-WR2")
 		(date "2025-07-16")
 		(rev "0.0.0")
