File: schematic/pslab-mini.kicad_sch (KiCad schematic)
At the start: 144 parts, among them J1 USB_C_Receptacle_USB2.0_16P, J2 Battery_Cell, J3 Conn_Coaxial, J4 Conn_Coaxial, J5 Conn_02x16_Odd_Even, J6 Conn_01x15_Socket, J7 Conn_02x03_Top_Bottom, Q1 MMBT3904, Q2 MMBT3906, SW1 Reset, SW2 Power, U1 MT2496, U10 TL082, U11 ESP32-C3, U2 AP3015A, U3 IP5189T, U4 SP0503BAHT, U5 AMS1117-3.3, U6 STM32H563RIT6, U7 TL082, U8 MCP6S21, U9 MCP6S21, X1 32kHz768, Y1 Crystal_25MHz, Y2 Crystal_40Mhz

Commit message: Update pslab-mini.kicad_sch
Other:
- title: PSLab-Mini -> PSLab-Mini-C
Changed lines of the file:
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@@
 	(paper "User" 586.969 296.977)
 	(title_block
-		(title "PSLab-Mini")
+		(title "PSLab-Mini-C")
 		(date "2025-07-16")
 		(rev "0.0.0")
